File: CH340G/CH340G.sch (KiCad schematic (older format))
At the start: 16 parts, among them J1 USB_B_Micro, J2 Conn_01x06, U1 CH340G, Y1 Crystal

Commit message: Power LED Added
Parts:
- removed C1, C2: 22pF, Capacitor_SMD:C_0805_2012Metric_Pad1.15x1.40mm_HandSolder, symbol Device:C
- removed JP1, JP2: SolderJumper_3_Bridged12, Jumper:SolderJumper-3_P1.3mm_Bridged12_RoundedPad1.0x1.5mm_NumberLabels, symbol Jumper:SolderJumper_3_Bridged12
- removed Y1: Crystal, Crystal:Crystal_SMD_2012-2Pin_2.0x1.2mm_HandSoldering, symbol Device:Crystal
- added C5: 10nF, Capacitor_SMD:C_0805_2012Metric_Pad1.15x1.40mm_HandSolder, symbol Device:C
- added JP1, JP2: SolderJumper_3_Open, Jumper:SolderJumper-3_P1.3mm_Open_RoundedPad1.0x1.5mm, symbol Jumper:SolderJumper_3_Open
- added PWR1: LED, LED_SMD:LED_0805_2012Metric_Castellated, symbol Device:LED
- added R3: R_US, Resistor_SMD:R_0805_2012Metric_Pad1.15x1.40mm_HandSolder, symbol Device:R_US
- added Y1: Resonator, Crystal:Resonator_SMD_muRata_CSTxExxV-3Pin_3.0x1.1mm, symbol Device:Resonator
- C3: value 10uF -> 22uF; footprint Capacitor_SMD:C_0805_2012Metric_Pad1.15x1.40mm_HandSolder -> Capacitor_Tantalum_SMD:CP_EIA-3216-18_Kemet-A_Pad1.58x1.35mm_HandSolder
- renumbered D3 to RX1, D4 to TX1
Connections:
- net labels added: VBUS
Other:
- moved on the sheet: J1
Changed lines of the file:
@@
 EESchema Schematic File Version 4
-LIBS:SirUSB-cache
 EELAYER 29 0
 EELAYER END
@@
 $EndComp
 $Comp
-L Device:LED D3
+L Device:LED RX1
 U 1 1 5D25DED7
 P 7300 2350
-F 0 "D3" H 7292 2564 50  0000 C CNN
+F 0 "RX1" H 7292 2564 50  0000 C CNN
 F 1 "LED" H 7292 2474 50  0000 C CNN
 F 2 "LED_SMD:LED_0805_2012Metric_Castellated" H 7300 2350 50  0001 C CNN
@@
 P 3500 3200
 F 0 "C3" H 3618 3245 50  0000 L CNN
-F 1 "10uF" H 3618 3155 50  0000 L CNN
-F 2 "Capacitor_SMD:C_0805_2012Metric_Pad1.15x1.40mm_HandSolder" H 3538 3050 50  0001 C CNN
+F 1 "22uF" H 3618 3155 50  0000 L CNN
+F 2 "Capacitor_Tantalum_SMD:CP_EIA-3216-18_Kemet-A_Pad1.58x1.35mm_HandSolder" H 3538 3050 50  0001 C CNN
 F 3 "~" H 3500 3200 50  0001 C CNN
 	1    3500 3200
 	1    0    0    -1
-$EndComp
-$Comp
-L Device:Crystal Y1
-U 1 1 5D25ECFD
-P 4850 3450
-F 0 "Y1" V 4895 3319 50  0000 R CNN
-F 1 "Crystal" V 4805 3319 50  0000 R CNN
-F 2 "Crystal:Crystal_SMD_2012-2Pin_2.0x1.2mm_HandSoldering" H 4850 3450 50  0001 C CNN
-F 3 "~" H 4850 3450 50  0001 C CNN
-	1    4850 3450
-	0    1    -1   0
 $EndComp
 $Comp
@@
 	1    0    0    -1
 $EndComp
-$Comp
-L Device:C C2
-U 1 1 5D260670
-P 4450 3200
-F 0 "C2" V 4700 3200 50  0000 C CNN
-F 1 "22pF" V 4610 3200 50  0000 C CNN
-F 2 "Capacitor_SMD:C_0805_2012Metric_Pad1.15x1.40mm_HandSolder" H 4488 3050 50  0001 C CNN
-F 3 "~" H 4450 3200 50  0001 C CNN
-	1    4450 3200
-	0    -1   -1   0
-$EndComp
-$Comp
-L Device:C C1
-U 1 1 5D260AF2
-P 4450 3700
-F 0 "C1" V 4700 3700 50  0000 C CNN
-F 1 "22pF" V 4610 3700 50  0000 C CNN
-F 2 "Capacitor_SMD:C_0805_2012Metric_Pad1.15x1.40mm_HandSolder" H 4488 3550 50  0001 C CNN
-F 3 "~" H 4450 3700 50  0001 C CNN
-	1    4450 3700
-	0    -1   1    0
-$EndComp
 Wire Wire Line
 	5200 3350 5200 3300
 Wire Wire Line
-	5200 3300 4850 3300
-Wire Wire Line
-	4600 3200 4600 3300
-Wire Wire Line
-	4600 3300 4850 3300
-Connection ~ 4850 3300
-Wire Wire Line
 	5200 3550 5200 3600
 Wire Wire Line
-	5200 3600 4850 3600
-Wire Wire Line
-	4850 3600 4600 3600
-Wire Wire Line
-	4600 3600 4600 3700
-Connection ~ 4850 3600
-Wire Wire Line
-	4300 3700 4200 3700
-Wire Wire Line
-	4200 3700 4200 3200
-Wire Wire Line
-	4200 3200 4300 3200
-Wire Wire Line
 	5600 3750 5600 4000
-Wire Wire Line
-	5600 4000 4200 4000
-Wire Wire Line
-	4200 4000 4200 3700
-Connection ~ 4200 3700
 $Comp
 L Connector:USB_B_Micro J1
 U 1 1 5D26FDA6
-P 3000 2700
-F 0 "J1" H 3056 3165 50  0000 C CNN
-F 1 "USB_B_Micro" H 3056 3075 50  0000 C CNN
-F 2 "Connector_USB:USB_Micro-B_Molex_47346-0001" H 3150 2650 50  0001 C CNN
-F 3 "~" H 3150 2650 50  0001 C CNN
-	1    3000 2700
+P 2650 2700
+F 0 "J1" H 2706 3165 50  0000 C CNN
+F 1 "USB_B_Micro" H 2706 3075 50  0000 C CNN
+F 2 "Connector_USB:USB_Micro-B_Molex_47346-0001" H 2800 2650 50  0001 C CNN
+F 3 "~" H 2800 2650 50  0001 C CNN
+	1    2650 2700
 	1    0    0    -1
 $EndComp
@@
 	5000 3050 5000 2700
 Wire Wire Line
-	5000 2700 3300 2700
-Wire Wire Line
-	3300 2800 4950 2800
+	5000 2700 2950 2700
+Wire Wire Line
+	2950 2800 4950 2800
 Wire Wire Line
 	4950 2800 4950 3150
@@
 	4950 3150 5200 3150
 Wire Wire Line
-	2900 3100 3000 3100
-Wire Wire Line
-	3000 3100 3000 4000
-Wire Wire Line
-	3000 4000 3500 4000
-Connection ~ 3000 3100
-Connection ~ 4200 4000
+	2550 3100 2650 3100
+Wire Wire Line
+	2650 3100 2650 4000
+Wire Wire Line
+	2650 4000 3150 4000
 Wire Wire Line
 	6000 2750 6450 2750
@@
 Wire Wire Line
 	6400 2850 6400 2950
-$Comp
-L Jumper:SolderJumper_3_Bridged12 JP2
-U 1 1 5D27956A
-P 6300 2400
-F 0 "JP2" H 6300 2603 50  0000 C CNN
-F 1 "SolderJumper_3_Bridged12" H 6300 2513 50  0000 C CNN
-F 2 "Jumper:SolderJumper-3_P1.3mm_Bridged12_RoundedPad1.0x1.5mm_NumberLabels" H 6300 2400 50  0001 C CNN
-F 3 "~" H 6300 2400 50  0001 C CNN
-	1    6300 2400
-	1    0    0    -1
-$EndComp
 Wire Wire Line
 	6000 3050 6100 3050
@@
 	6700 3250 6700 4000
 Wire Wire Line
-	6650 3050 6650 2300
-Wire Wire Line
-	6650 2300 5600 2300
-$Comp
-L Device:LED D4
+	6650 1850 5600 1850
+$Comp
+L Device:LED TX1
 U 1 1 5D284AF1
 P 7650 2350
-F 0 "D4" H 7642 2564 50  0000 C CNN
+F 0 "TX1" H 7642 2564 50  0000 C CNN
 F 1 "LED" H 7642 2474 50  0000 C CNN
 F 2 "LED_SMD:LED_0805_2012Metric_Castellated" H 7650 2350 50  0001 C CNN
@@
 	6650 1550 7300 1550
 Wire Wire Line
-	6650 1550 6650 2300
-Connection ~ 6650 2300
+	6650 1550 6650 1850
 Connection ~ 7300 1550
-Text Label 5750 2300 0    50   ~ 0
+Text Label 5750 1850 0    50   ~ 0
 5V
 Text Label 6000 4000 0    50   ~ 0
@@
 Connection ~ 3500 2500
 Wire Wire Line
-	3500 2500 3300 2500
+	3500 2500 3150 2500
 Wire Wire Line
 	3850 3050 3850 2500
@@
 Connection ~ 3850 4000
 Wire Wire Line
-	3850 4000 4200 4000
+	3850 4000 4050 4000
 Text Label 4650 2700 0    50   ~ 0
 D+
@@
 Wire Wire Line
 	4250 2050 4450 2050
-$Comp
-L Jumper:SolderJumper_3_Bridged12 JP1
-U 1 1 5D26E52F
-P 4850 1650
-F 0 "JP1" H 4850 1853 50  0000 C CNN
-F 1 "SolderJumper_3_Bridged12" H 4850 1763 50  0000 C CNN
-F 2 "Jumper:SolderJumper-3_P1.3mm_Bridged12_RoundedPad1.0x1.5mm_NumberLabels" H 4850 1650 50  0001 C CNN
-F 3 "~" H 4850 1650 50  0001 C CNN
-	1    4850 1650
-	1    0    0    -1
-$EndComp
 Wire Wire Line
 	3850 2050 3850 1650
-Wire Wire Line
-	3850 1650 4650 1650
 Connection ~ 3850 2050
-Wire Wire Line
-	4850 1800 4850 2050
-Wire Wire Line
-	4850 2050 4750 2050
-Wire Wire Line
-	5600 2300 5600 2550
-Wire Wire Line
-	4850 2050 5600 2050
-Wire Wire Line
-	5600 2050 5600 2300
-Connection ~ 4850 2050
-Connection ~ 5600 2300
-Wire Wire Line
-	5050 1650 5500 1650
-Wire Wire Line
-	5500 1650 5500 2550
+$Comp
+L Device:LED PWR1
+U 1 1 5D61F292
+P 3150 3450
+F 0 "PWR1" H 3142 3664 50  0000 C CNN
+F 1 "LED" H 3142 3574 50  0000 C CNN
+F 2 "LED_SMD:LED_0805_2012Metric_Castellated" H 3150 3450 50  0001 C CNN
+F 3 "~" H 3150 3450 50  0001 C CNN
+	1    3150 3450
+	0    -1   -1   0
+$EndComp
+$Comp
+L Device:R_US R3
+U 1 1 5D61F298
+P 3150 3050
+F 0 "R3" H 3218 3095 50  0000 L CNN
+F 1 "R_US" H 3218 3005 50  0000 L CNN
+F 2 "Resistor_SMD:R_0805_2012Metric_Pad1.15x1.40mm_HandSolder" V 3190 3040 50  0001 C CNN
+F 3 "~" H 3150 3050 50  0001 C CNN
+	1    3150 3050
+	1    0    0    -1
+$EndComp
+Wire Wire Line
+	3150 3300 3150 3200
+Connection ~ 2650 3100
+Wire Wire Line
+	3150 2500 3150 2900
+Connection ~ 3150 2500
+Wire Wire Line
+	3150 2500 2950 2500
+Wire Wire Line
+	3150 3600 3150 4000
+Connection ~ 3150 4000
+Wire Wire Line
+	3150 4000 3500 4000
+$Comp
+L Jumper:SolderJumper_3_Open JP1
+U 1 1 5D65075B
+P 5000 1850
+F 0 "JP1" H 5000 1963 50  0000 C CNN
+F 1 "SolderJumper_3_Open" H 5000 1963 50  0001 C CNN
+F 2 "Jumper:SolderJumper-3_P1.3mm_Open_RoundedPad1.0x1.5mm" H 5000 1850 50  0001 C CNN
+F 3 "~" H 5000 1850 50  0001 C CNN
+	1    5000 1850
+	0    -1   -1   0
+$EndComp
+$Comp
+L Jumper:SolderJumper_3_Open JP2
+U 1 1 5D651B6F
+P 6300 2400
+F 0 "JP2" H 6300 2513 50  0000 C CNN
+F 1 "SolderJumper_3_Open" H 6300 2513 50  0001 C CNN
+F 2 "Jumper:SolderJumper-3_P1.3mm_Open_RoundedPad1.0x1.5mm" H 6300 2400 50  0001 C CNN
+F 3 "~" H 6300 2400 50  0001 C CNN
+	1    6300 2400
+	1    0    0    -1
+$EndComp
+Text Label 3850 1650 0    50   ~ 0
+VBUS
+Wire Wire Line
+	4750 2050 5000 2050
+$Comp
+L Device:C C5
+U 1 1 5D66AAEE
+P 4900 2300
+F 0 "C5" V 5150 2300 50  0000 C CNN
+F 1 "10nF" V 5060 2300 50  0000 C CNN
+F 2 "Capacitor_SMD:C_0805_2012Metric_Pad1.15x1.40mm_HandSolder" H 4938 2150 50  0001 C CNN
+F 3 "~" H 4900 2300 50  0001 C CNN
+	1    4900 2300
+	0    -1   1    0
+$EndComp
+Wire Wire Line
+	5050 2300 5500 2300
+Wire Wire Line
+	5500 2300 5500 2550
+Wire Wire Line
+	4750 2300 4050 2300
+Wire Wire Line
+	4050 2300 4050 4000
+Connection ~ 4050 4000
+Wire Wire Line
+	3850 1650 5000 1650
+Wire Wire Line
+	5150 1850 5600 1850
+Connection ~ 5600 1850
+Connection ~ 6650 1850
+Wire Wire Line
+	6650 1850 6650 3050
+Wire Wire Line
+	5600 1850 5600 2550
+$Comp
+L Device:Resonator Y1
+U 1 1 5D69C84F
+P 4900 3450
+F 0 "Y1" V 4855 3561 50  0000 L CNN
+F 1 "Resonator" V 4945 3561 50  0000 L CNN
+F 2 "Crystal:Resonator_SMD_muRata_CSTxExxV-3Pin_3.0x1.1mm" H 4875 3450 50  0001 C CNN
+F 3 "~" H 4875 3450 50  0001 C CNN
+	1    4900 3450
+	0    1    -1   0
+$EndComp
+Wire Wire Line
+	4900 3300 5200 3300
+Wire Wire Line
+	4900 3600 5200 3600
+Wire Wire Line
+	4050 4000 4500 4000
+Wire Wire Line
+	4700 3450 4500 3450
+Wire Wire Line
+	4500 3450 4500 4000
+Connection ~ 4500 4000
+Wire Wire Line
+	4500 4000 5600 4000
 $EndSCHEMATC

Commit message: Page Settings Updated
Parts:
- R1, R2, R3: value R_US -> 470E
Other:
- moved on the sheet: C3, C4, C5, D1, D2, J1, J2, JP1, JP2, PWR1, R1, R2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

Commit message: CH340G Revision 2
Parts:
- removed D1, D2: D, Diode_SMD:D_MiniMELF, symbol Device:D
- removed J1: USB_B_Micro, Connector_USB:USB_Micro-B_Molex_47346-0001, symbol Connector:USB_B_Micro
- removed TX1: LED, LED_SMD:LED_0805_2012Metric_Castellated, symbol Device:LED
- removed Y1: Resonator, Crystal:Resonator_SMD_muRata_CSTxExxV-3Pin_3.0x1.1mm, symbol Device:Resonator
- added C1, C2: 9pF, Capacitor_SMD:C_0603_1608Metric, symbol Device:C
- added C6, C7: 10uF, Capacitor_SMD:C_0805_2012Metric, symbol Device:C
- added D1: PRTR5V0U2X, Package_TO_SOT_SMD:SOT-143, symbol Power_Protection:PRTR5V0U2X
- added F1: 500mA, Resistor_SMD:R_0805_2012Metric, symbol Device:Fuse
- added P1: USB_C_Plug_USB2.0, SirBoardLibrary:USB_C, symbol SirBoard_Library:USB_C_Plug_USB2.0
- added TX2: RED, LED_SMD:LED_0603_1608Metric, symbol Device:LED
- added U2: AP2127K-3.3, Package_TO_SOT_SMD:SOT-23-5, symbol Regulator_Linear:AP2127K-3.3
- added Y1: Crystal_GND24, Crystal:Crystal_SMD_SeikoEpson_TSX3225-4Pin_3.2x2.5mm, symbol Device:Crystal_GND24
- C3: Part (none) -> C122643
- C4: footprint Capacitor_SMD:C_0805_2012Metric_Pad1.15x1.40mm_HandSolder -> Capacitor_SMD:C_0603_1608Metric; Part (none) -> C42998
- C5: footprint Capacitor_SMD:C_0805_2012Metric_Pad1.15x1.40mm_HandSolder -> Capacitor_SMD:C_0603_1608Metric; Part (none) -> C100042
- PWR1: value LED -> BLUE; footprint LED_SMD:LED_0805_2012Metric_Castellated -> LED_SMD:LED_0603_1608Metric; Part (none) -> C193191
- R1, R2: value 470E -> 1K; footprint Resistor_SMD:R_0805_2012Metric_Pad1.15x1.40mm_HandSolder -> Resistor_SMD:R_0603_1608Metric; Part (none) -> C269441
- R3: value 470E -> 1K; footprint Resistor_SMD:R_0805_2012Metric_Pad1.15x1.40mm_HandSolder -> Resistor_SMD:R_0603_1608Metric; Part (none) -> C25585
- RX1: value LED -> GREEN; footprint LED_SMD:LED_0805_2012Metric_Castellated -> LED_SMD:LED_0603_1608Metric; Part (none) -> C205443
Connections:
- net CTS: now also J2.5 (Pin_5); no longer JP2.1 (A)
- net D+: now also D1.2 (I/O1), P1.A6 (D+), P1.B6 (D+)
- net D-: now also D1.3 (I/O2), P1.A7 (D-), P1.B7 (D-)
- net DTR: now also JP2.1 (A); no longer J2.1 (Pin_1)
- net GND: now also RX1.1 (K), C1.2, C2.2, C6.2, C7.2, D1.1 (GND), P1.A1 (GND), P1.A12 (GND), P1.B1 (GND), P1.B12 (GND), P1.S1 (SHIELD), TX2.1 (K), U2.2 (GND), Y1.2, Y1.4
- net RX: now also R3.1, U1.3 (RXD); no longer RX1.1 (K), U1.2 (TXD)
- net TX: now also R2.1, U1.2 (TXD); no longer U1.3 (RXD)
- net VBUS: now also JP1.1 (A), C6.1, D1.4 (VCC), F1.1, U2.1 (VIN), U2.3 (EN); no longer JP1.3 (B), R3.1
- net 3V3: now reaches C5.2, U1.4 (V3)
- net 3V3: now also JP1.3 (B), C7.1, U2.5 (VOUT)
- net at U1.7 (XI): now also C1.1, Y1.1
- net at U1.8 (XO): now also C2.1, Y1.3
- net at RX1.2 (A): now also R3.2; no longer R1.2
- net at R2.2: now also TX2.2 (A)
- net at PWR1.2 (A): now also R1.2; no longer R3.2
- net 5V renamed VCC
- net VCC: no longer R2.1
- net R_C renamed P6
- net P6: now also J2.1 (Pin_1); no longer J2.5 (Pin_5)
- new net: F1.2, P1.A4 (VBUS), P1.A9 (VBUS), P1.B4 (VBUS), P1.B9 (VBUS)
Other:
- moved on the sheet: C3, C4, C5, J2, JP1, JP2, U1
