File: FT230/FT230.kicad_pcb (KiCad board)
At the start: 2 copper layers, 21.1 x 10.4 mm, 22 parts, among them J1 USB_B_Micro, J2 Conn_01x04, J3 Conn_01x02, J4 Conn_01x02, U1 FT230XQ

Commit message: Soldermask width adjusted
Other:
- rule solder_mask_min_width: 0.1 -> 0.05
Changed lines of the file:
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@@
     (pad_drill 1)
     (pad_to_mask_clearance 0)
-    (solder_mask_min_width 0.1)
+    (solder_mask_min_width 0.05)
     (aux_axis_origin 0 0)
     (visible_elements 7FFFFFFF)
