File: CP2104/CP2104.sch (KiCad schematic (older format))
At the start: 17 parts, among them J1 Conn_01x06, P1 USB_C_Plug_USB2.0, U1 CP2104

Commit message: SirUSB Board Revisions
Removed MicroUSB Versions of FT230 and FT231, SolderPaste Layer Adjusted to -0.05mm, Silkscreens optimised, OSHW logo added.
Parts:
- U1: Part (none) -> C47742
Changed lines of the file:
@@
 F 2 "Package_DFN_QFN:QFN-24-1EP_4x4mm_P0.5mm_EP2.6x2.6mm" H 4925 900 50  0001 L CNN
 F 3 "https://www.silabs.com/documents/public/data-sheets/cp2104.pdf" H 4225 3100 50  0001 C CNN
+F 4 "C47742" H 4775 1850 50  0001 C CNN "Part"
 	1    4775 1850
 	1    0    0    -1
